File: robot-encoder-module/robot-encoder-module.kicad_sch (KiCad schematic)
At the start: 14 parts, among them J1 Conn_02x12_Odd_Even, U1 LS7366R, U2 LS7366R, U3 LS7366R, U4 LS7366R, U5 LS7366R, U6 LS7366R, X1 ABLS-20.000MHZ-B2-T

Commit message: Schematic Tweaks and Board stackup
Tweaks to scheamtic and creation of board stackup.
Parts:
- added C7: C0805C104M5RACTU, AVR-KiCAD-Lib-Capacitors:C0805, symbol AVR-KiCAD-Lib-Capacitors:C0805C104M5RACTU
- added U7: SN74LVC1G14DBV, Package_TO_SOT_SMD:SOT-23-5, symbol 74xGxx:SN74LVC1G14DBV
Connections:
- net +3V3: now also C7.2, U7.5 (VCC)
- net GND: now also C7.1, U7.3 (GND)
- net XTAL: now reaches U1.1 (fCKO), X1.1
- net XTAL: now also U7.2
- net CLOCK: now reaches U4.2 (fCKi)
- net CLOCK: now also U2.2 (fCKi), U3.2 (fCKi), U5.2 (fCKi), U6.2 (fCKi), U7.4
